File: Shield_PAMI/Shield_PAMI.kicad_sch (KiCad schematic)
At the start: 0 parts

Commit message: Fin creation du shield
Parts:
- added H1, H2, H3, H4: MountingHole_Pad, MountingHole:MountingHole_2.2mm_M2_Pad_TopBottom, symbol Mechanical:MountingHole_Pad
- added J1: Conn_01x02, Connector_JST:JST_XH_B2B-XH-AM_1x02_P2.50mm_Vertical, symbol Connector_Generic:Conn_01x02
- added J2, J3: Conn_01x06, Connector_JST:JST_XH_B6B-XH-AM_1x06_P2.50mm_Vertical, symbol Connector_Generic:Conn_01x06
- added J4: Conn_01x04, Connector_JST:JST_XH_B4B-XH-AM_1x04_P2.50mm_Vertical, symbol Connector_Generic:Conn_01x04
- added U1: NUCLEO-L476RG, NUCLEO-L476RG:MODULE_NUCLEO-L476RG, symbol NUCLEO-L476RG:NUCLEO-L476RG
- added U2: L293D, L293D:DIP880W50P254L2000H510Q16, symbol L293D:L293D
Connections:
- new net +3V3: J2.5 (Pin_5), J3.5 (Pin_5), J4.1 (Pin_1), U1.CN7_16 (+3V3)
- new net +6V: J1.2 (Pin_2), U1.CN7_24 (VIN), U2.16 (VSS), U2.8 (VS)
- new net EN1: U1.CN7_28 (PA0), U2.1 (ENABLE1)
- new net EN2: U1.CN7_30 (PA1), U2.9 (ENABLE2)
- new net Echo: J4.2 (Pin_2), U1.CN7_3 (PC12)
- new net GND: H1.1, H2.1, H3.1, H4.1, J1.1 (Pin_1), J2.2 (Pin_2), J3.2 (Pin_2), J4.4 (Pin_4), U1.CN10_20 (GND_CN10_20), U1.CN10_32 (AGND), U1.CN10_9 (GND_CN10_9), U1.CN7_19 (GND_CN7_19), U1.CN7_20 (GND_CN7_20), U1.CN7_22 (GND_CN7_22), U1.CN7_8 (GND_CN7_8), U2.12 (GND), U2.13 (GND), U2.4 (GND), U2.5 (GND)
- new net IN1: U1.CN7_35 (PC2), U2.2 (INPUT1)
- new net IN2: U1.CN7_37 (PC3), U2.7 (INPUT2)
- new net IN3: U1.CN7_38 (PC0), U2.10 (INPUT3)
- new net IN4: U1.CN7_36 (PC1), U2.15 (INPUT4)
- new net Out1: J2.1 (Pin_1), U2.3 (OUTPUT1)
- new net Out2: J2.6 (Pin_6), U2.6 (OUTPUT2)
- new net Out3: J3.1 (Pin_1), U2.11 (OUTPUT3)
- new net Out4: J3.6 (Pin_6), U2.14 (OUTPUT4)
- new net Trig: J4.3 (Pin_3), U1.CN7_1 (PC10)
- new net left_enc_A: J2.3 (Pin_3), U1.CN10_13 (PA6)
- new net left_enc_B: J2.4 (Pin_4), U1.CN10_15 (PA7)
- new net right_enc_A: J3.3 (Pin_3), U1.CN10_23 (PA8)
- new net right_enc_B: J3.4 (Pin_4), U1.CN10_21 (PA9)
- no-connect marks 0 -> 48
Other:
- note added: "MOTOR1"
- note added: "MOTOR2"
- note added: "ULTRA-SOUND"
